File: design.kicad_pcb (KiCad board)
At the start: 2 copper layers, 0 parts

Commit message: initial commit
Parts:
- added C1: C_Small, Capacitor_SMD:C_0805_2012Metric, F.Cu at (150.5, 83.0)
- added C2: C_Small, Capacitor_SMD:C_0805_2012Metric, F.Cu at (154.9, 83.0)
- added J1: USB_C_Receptacle, Connector_USB:USB_C_Receptacle_HRO_TYPE-C-31-M-12, F.Cu at (140.5, 86.0)
- added J2: Conn_01x05, E32-xxxT20D:UDPI_interface, F.Cu at (161.5, 85.5)
- added U1: ATtiny1616-M, Package_DFN_QFN:VQFN-20-1EP_3x3mm_P0.4mm_EP1.7x1.7mm, F.Cu at (152.6, 88.5)
Other:
- board outline added: 28.5 x 12 mm

Commit message: add hash label
Other:
- board text added: "<<hash>>"
Changed lines of the file:
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@@
   (general
     (thickness 1.6)
-    (drawings 4)
+    (drawings 5)
     (tracks 0)
     (zones 0)
@@
     )
   )
+  (gr_text <<hash>> (at 160 90.5) (layer F.SilkS)
+    (effects (font (size 1 1) (thickness 0.15)))
+  )
   (gr_line (start 136.5 92) (end 136.5 80) (layer Edge.Cuts) (width 0.05))
