File: design.kicad_pcb (KiCad board)
At the start: 2 copper layers, 28.5 x 12 mm, 5 parts, among them J1 USB_C_Receptacle, J2 Conn_01x05, U1 ATtiny1616-M

Commit message: add LED
Parts:
- added D1: LED, LED_THT:LED_D5.0mm_FlatTop, F.Cu at (148.0, 88.3)
- moved U1 2.95 mm to (155.5, 88.5)

Commit message: add LED
Parts:
- added D2: LED, LED_SMD:LED_0603_1608Metric_Pad1.05x0.95mm_HandSolder, F.Cu at (158.1, 81.0)

Commit message: add text
Other:
- board text added: "<<date>>"
- board text added: "<<project_name>>"
- board text added: "<<version>>"
