File: design.kicad_pcb (KiCad board)
At the start: 2 copper layers, 25 x 22.9 mm, 14 parts, among them J1 Conn_01x02, J2 Conn_01x02, J3 Conn_01x03, J4 Conn_01x03, U1 TPS61099YFFT

Commit message: fake change
Routing:
- net GND: vias 35 -> 36
Changed lines of the file:
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@@
   (via (at 140.716 90.17) (size 0.8) (drill 0.4) (layers "F.Cu" "B.Cu") (free) (net 2))
   (via (at 152.908 104.648) (size 0.8) (drill 0.4) (layers "F.Cu" "B.Cu") (free) (net 2))
+  (via (at 157 99.75) (size 0.8) (drill 0.4) (layers "F.Cu" "B.Cu") (free) (net 2))
   (via (at 152.908 88.138) (size 0.8) (drill 0.4) (layers "F.Cu" "B.Cu") (free) (net 2))
   (via (at 154.178 103.378) (size 0.8) (drill 0.4) (layers "F.Cu" "B.Cu") (free) (net 2))

Commit message: fake change
Routing:
- net GND: vias 36 -> 35
Changed lines of the file:
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@@
   (via (at 136.906 90.17) (size 0.8) (drill 0.4) (layers "F.Cu" "B.Cu") (free) (net 2))
   (via (at 139.446 91.44) (size 0.8) (drill 0.4) (layers "F.Cu" "B.Cu") (free) (net 2))
-  (via (at 157.25 102.25) (size 0.8) (drill 0.4) (layers "F.Cu" "B.Cu") (free) (net 2))
   (via (at 140.716 90.17) (size 0.8) (drill 0.4) (layers "F.Cu" "B.Cu") (free) (net 2))
   (via (at 152.908 104.648) (size 0.8) (drill 0.4) (layers "F.Cu" "B.Cu") (free) (net 2))
