File: design.sch (KiCad schematic (older format))
At the start: 5 parts, among them J1 USB_C_Receptacle, J2 Conn_01x05, U1 ATtiny1616-M

Commit message: add LED
Parts:
- added D1: LED, LED_THT:LED_D5.0mm_FlatTop, symbol Device:LED
Changed lines of the file:
@@
+	1    0    0    -1
+$EndComp
+$Comp
+L Device:LED D1
+U 1 1 61E9317C
+P 6900 4600
+F 0 "D1" H 6893 4817 50  0000 C CNN
+F 1 "LED" H 6893 4726 50  0000 C CNN
+F 2 "LED_THT:LED_D5.0mm_FlatTop" H 6900 4600 50  0001 C CNN
+F 3 "~" H 6900 4600 50  0001 C CNN
+	1    6900 4600
 	1    0    0    -1
 $EndComp

Commit message: add LED
Parts:
- added D2: LED, LED_SMD:LED_0603_1608Metric_Pad1.05x0.95mm_HandSolder, symbol Device:LED
Changed lines of the file:
@@
+	1    0    0    -1
+$EndComp
+$Comp
+L Device:LED D2
+U 1 1 61E9D790
+P 7500 4600
+F 0 "D2" H 7493 4817 50  0000 C CNN
+F 1 "LED" H 7493 4726 50  0000 C CNN
+F 2 "LED_SMD:LED_0603_1608Metric_Pad1.05x0.95mm_HandSolder" H 7500 4600 50  0001 C CNN
+F 3 "~" H 7500 4600 50  0001 C CNN
+	1    7500 4600
 	1    0    0    -1
 $EndComp
