File: design.kicad_sch (KiCad schematic)
At the start: 14 parts, among them J1 Conn_01x02, J2 Conn_01x02, J3 Conn_01x03, J4 Conn_01x03, U1 TPS61099YFFT

Commit message: ADD ID to SCH&PCB Page
Other:
- title: <<project_name>> -> <<ID>>_<<project_name>>
Changed lines of the file:
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@@
   (paper "A4")
   (title_block
-    (title "<<project_name>>")
+    (title "<<ID>>_<<project_name>>")
     (date "<<date>>")
     (rev "<<version>>")
