File: PFFF.kicad_pcb (KiCad board)
At the start: 2 copper layers, 25 x 22.9 mm, 14 parts, among them J1 Conn_01x02, J2 Conn_01x02, J3 Conn_01x03, J4 Conn_01x03, U1 TPS61099YFFT

Commit message: Update Bom and PCB_top
Other:
- board text added: "template ID:PFFF <<version>> 2024-06-02 Git-0d2bf0b www.website.com//PFFF"
- board text removed: "<<project_name>> <<ID>> <<version>> <<date>> <<hash>> <<website_link>>"
Changed lines of the file:
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@@
 	(paper "A4")
 	(title_block
-		(title "<<ID>>_<<project_name>>")
-		(date "<<date>>")
+		(title "ID:PFFF_template")
+		(date "2024-06-02")
 		(rev "<<version>>")
-		(comment 4 "<<hash>>")
+		(comment 4 "Git-0d2bf0b")
 	)
 	(layers
@@
 		(layer "Edge.Cuts")
 	)
-	(gr_text "<<project_name>>\n<<ID>>\n<<version>>\n<<date>>\n<<hash>>\n<<website_link>>"
+	(gr_text "template\nID:PFFF\n<<version>>\n2024-06-02\nGit-0d2bf0b\nwww.website.com//PFFF"
 		(at 146.5 95.504 0)
 		(layer "B.SilkS")
@@
 		)
 	)
-	(gr_text "<<project_name>>\n<<ID>>\n<<version>>\n<<date>>\n<<hash>>\n<<website_link>>"
+	(gr_text "template\nID:PFFF\n<<version>>\n2024-06-02\nGit-0d2bf0b\nwww.website.com//PFFF"
 		(at 225.75 151 0)
 		(layer "F.SilkS")
