File: PFFF.kicad_sch (KiCad schematic)
At the start: 14 parts, among them J1 Conn_01x02, J2 Conn_01x02, J3 Conn_01x03, J4 Conn_01x03, U1 TPS61099YFFT

Commit message: Update Bom and PCB_top
Other:
- title: <<ID>>_<<project_name>> -> PFFF_template
Changed lines of the file:
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@@
 	(paper "A4")
 	(title_block
-		(title "<<ID>>_<<project_name>>")
-		(date "<<date>>")
+		(title "PFFF_template")
+		(date "2024-06-02")
 		(rev "<<version>>")
-		(comment 4 "<<hash>>")
+		(comment 4 "Git-0d2bf0b")
 	)
 	(junction
